File: 50x50_bottom_left.sch (KiCad schematic (older format))
At the start: 98 parts, among them CON1 BARREL_JACK, J1 INTERCONNECT_1X03, J10 INTERCONNECT_1X03, J11 INTERCONNECT_1X03, J12 INTERCONNECT_1X03, J13 INTERCONNECT_1X03, J14 INTERCONNECT_1X03, J15 INTERCONNECT_1X03, J16 INTERCONNECT_1X03, J17 INTERCONNECT_1X03, J18 INTERCONNECT_1X03, J19 INTERCONNECT_1X03, J2 INTERCONNECT_1X03, J20 INTERCONNECT_1X03, J21 INTERCONNECT_1X03, J22 INTERCONNECT_1X03, J23 INTERCONNECT_1X03, J24 INTERCONNECT_1X03, J25 INTERCONNECT_1X03, J26 INTERCONNECT_1X03, J27 INTERCONNECT_1X03, J28 INTERCONNECT_1X03, J29 INTERCONNECT_1X03, J3 INTERCONNECT_1X03, J30 INTERCONNECT_1X03, J31 INTERCONNECT_1X03, J32 INTERCONNECT_1X03, J33 INTERCONNECT_1X03, J34 INTERCONNECT_1X03, J35 INTERCONNECT_1X03, J36 INTERCONNECT_1X03, J37 INTERCONNECT_1X03, J38 INTERCONNECT_1X03, J39 INTERCONNECT_1X03, J4 INTERCONNECT_1X03, J40 INTERCONNECT_1X03, J41 INTERCONNECT_1X03, J42 INTERCONNECT_1X03, J43 INTERCONNECT_1X03, J44 INTERCONNECT_1X03, J45 INTERCONNECT_1X03, J46 INTERCONNECT_1X03, J47 INTERCONNECT_1X03, J48 INTERCONNECT_1X03, J49 INTERCONNECT_1X03, J5 INTERCONNECT_1X03, J50 INTERCONNECT_1X03, J51 INTERCONNECT_1X03, J52 INTERCONNECT_1X03, J53 INTERCONNECT_1X03, J54 INTERCONNECT_1X03, J55 INTERCONNECT_1X03, J56 INTERCONNECT_1X03, J57 INTERCONNECT_1X03, J58 INTERCONNECT_1X03, J59 INTERCONNECT_1X03, J6 INTERCONNECT_1X03, J60 INTERCONNECT_1X03, J61 INTERCONNECT_1X03, J62 INTERCONNECT_1X03, J63 INTERCONNECT_1X03, J64 INTERCONNECT_1X03, J65 INTERCONNECT_1X02, J7 INTERCONNECT_1X03, J8 INTERCONNECT_1X03, J9 INTERCONNECT_1X03, P1 CONN_6X2, P2 CONN_6X2, U1 LM7805CT

Commit message: increased .1" edge connector from 2*6 to 2*8 to account for the A-100 system bus used in modular synthesizers
Parts:
- P1, P2: value CONN_6X2 -> CONN_8X2; symbol CONN_6X2 -> CONN_8X2
Connections:
- new net: P1.13, P2.13
- new net: P1.14, P2.14
- new net: P1.15, P2.15
- new net: P1.16, P2.16
Changed lines of the file:
@@
 $EndComp
 $Comp
-L CONN_6X2 P1
+L CONN_8X2 P1
 U 1 1 554C2B9D
-P 2100 3200
-F 0 "P1" H 2100 3550 60  0000 C CNN
-F 1 "CONN_6X2" V 2100 3200 60  0000 C CNN
-F 2 "" H 2100 3200 60  0000 C CNN
-F 3 "" H 2100 3200 60  0000 C CNN
-	1    2100 3200
+P 1950 3100
+F 0 "P1" H 1950 3450 60  0000 C CNN
+F 1 "CONN_8X2" V 1950 3100 60  0000 C CNN
+F 2 "" H 1950 3100 60  0000 C CNN
+F 3 "" H 1950 3100 60  0000 C CNN
+	1    1950 3100
 	1    0    0    1
 $EndComp
 $Comp
-L CONN_6X2 P2
+L CONN_8X2 P2
 U 1 1 554C2C4F
-P 2100 4000
-F 0 "P2" H 2100 4350 60  0000 C CNN
-F 1 "CONN_6X2" V 2100 4000 60  0000 C CNN
-F 2 "" H 2100 4000 60  0000 C CNN
-F 3 "" H 2100 4000 60  0000 C CNN
-	1    2100 4000
+P 1950 4100
+F 0 "P2" H 1950 4450 60  0000 C CNN
+F 1 "CONN_8X2" V 1950 4100 60  0000 C CNN
+F 2 "" H 1950 4100 60  0000 C CNN
+F 3 "" H 1950 4100 60  0000 C CNN
+	1    1950 4100
 	1    0    0    -1
 $EndComp
@@
 	3850 4500 3900 4500
 Wire Wire Line
-	1700 3450 1700 3750
-Wire Wire Line
-	2500 3450 2500 3750
-Wire Wire Line
-	2500 3350 2550 3350
-Wire Wire Line
-	2550 3350 2550 3850
-Wire Wire Line
-	2550 3850 2500 3850
-Wire Wire Line
-	2500 3250 2600 3250
-Wire Wire Line
-	2600 3250 2600 3950
-Wire Wire Line
-	2600 3950 2500 3950
-Wire Wire Line
-	2500 3150 2650 3150
-Wire Wire Line
-	2650 3150 2650 4050
-Wire Wire Line
-	2650 4050 2500 4050
-Wire Wire Line
-	2500 3050 2700 3050
-Wire Wire Line
-	2700 3050 2700 4150
-Wire Wire Line
-	2700 4150 2500 4150
-Wire Wire Line
-	2500 2950 2750 2950
-Wire Wire Line
-	2750 2950 2750 4250
-Wire Wire Line
-	2750 4250 2500 4250
-Wire Wire Line
-	1700 3350 1650 3350
-Wire Wire Line
-	1650 3350 1650 3850
-Wire Wire Line
-	1650 3850 1700 3850
-Wire Wire Line
-	1700 3250 1600 3250
-Wire Wire Line
-	1600 3250 1600 3950
-Wire Wire Line
-	1600 3950 1700 3950
-Wire Wire Line
-	1700 3150 1550 3150
-Wire Wire Line
-	1550 3150 1550 4050
-Wire Wire Line
-	1550 4050 1700 4050
-Wire Wire Line
-	1700 3050 1500 3050
-Wire Wire Line
-	1500 3050 1500 4150
-Wire Wire Line
-	1500 4150 1700 4150
-Wire Wire Line
-	1700 2950 1450 2950
-Wire Wire Line
-	1450 2950 1450 4250
-Wire Wire Line
-	1450 4250 1700 4250
+	1550 3450 1550 3750
+Wire Wire Line
+	2350 3450 2350 3750
+Wire Wire Line
+	2350 3350 2400 3350
+Wire Wire Line
+	2400 3350 2400 3850
+Wire Wire Line
+	2400 3850 2350 3850
+Wire Wire Line
+	2350 3250 2450 3250
+Wire Wire Line
+	2450 3250 2450 3950
+Wire Wire Line
+	2450 3950 2350 3950
+Wire Wire Line
+	2350 3150 2500 3150
+Wire Wire Line
+	2500 3150 2500 4050
+Wire Wire Line
+	2500 4050 2350 4050
+Wire Wire Line
+	2350 3050 2550 3050
+Wire Wire Line
+	2550 3050 2550 4150
+Wire Wire Line
+	2550 4150 2350 4150
+Wire Wire Line
+	2350 2950 2600 2950
+Wire Wire Line
+	2600 2950 2600 4250
+Wire Wire Line
+	2600 4250 2350 4250
+Wire Wire Line
+	1550 3350 1500 3350
+Wire Wire Line
+	1500 3350 1500 3850
+Wire Wire Line
+	1500 3850 1550 3850
+Wire Wire Line
+	1550 3250 1450 3250
+Wire Wire Line
+	1450 3250 1450 3950
+Wire Wire Line
+	1450 3950 1550 3950
+Wire Wire Line
+	1550 3150 1400 3150
+Wire Wire Line
+	1400 3150 1400 4050
+Wire Wire Line
+	1400 4050 1550 4050
+Wire Wire Line
+	1550 3050 1350 3050
+Wire Wire Line
+	1350 3050 1350 4150
+Wire Wire Line
+	1350 4150 1550 4150
+Wire Wire Line
+	1550 2950 1300 2950
+Wire Wire Line
+	1300 2950 1300 4250
+Wire Wire Line
+	1300 4250 1550 4250
+Wire Wire Line
+	2350 2850 2650 2850
+Wire Wire Line
+	2650 2850 2650 4350
+Wire Wire Line
+	2650 4350 2350 4350
+Wire Wire Line
+	2350 4450 2700 4450
+Wire Wire Line
+	2700 4450 2700 2750
+Wire Wire Line
+	2700 2750 2350 2750
+Wire Wire Line
+	1550 2850 1250 2850
+Wire Wire Line
+	1250 2850 1250 4350
+Wire Wire Line
+	1250 4350 1550 4350
+Wire Wire Line
+	1550 4450 1200 4450
+Wire Wire Line
+	1200 4450 1200 2750
+Wire Wire Line
+	1200 2750 1550 2750
 $EndSCHEMATC
